Commit message: adds gazebo model and control package
The model is made compatible with Gazebo.
Transmission tags are added and the joint positions can be controlled
and visualized in Gazebo.

File: robot/kai_description/urdf/geometry.xacro (robot description, xacro)
@@ -19,4 +19,5 @@
       depth="${base_platform_depth}" height="${base_platform_height}" />
   </link>
+  <!--JOINT Base_fixed-->
   <joint name="base_fixed_joint" type="fixed">
     <parent link="base_platform_link" />
@@ -25,4 +26,5 @@
     <origin xyz="0 0 ${base_platform_height}" rpy="0 0 0"/>
   </joint>
+  <!--Base Cylinder-->
   <link name="base_cylinder_link">
     <collision>
@@ -41,4 +43,5 @@
     <xacro:cylinder_center_inertia mass="${base_cylinder_mass}" radius="${base_cylinder_radius}" length="${base_cylinder_length}" />
   </link>
+  <!--JOINT Base_pole-->
   <joint name="base_pole_joint" type="continuous">
     <parent link="base_cylinder_link" />
@@ -47,4 +50,5 @@
     <axis xyz="0 0 1" />
   </joint>
+ <!--Pole-->
  <link name="pole_link">
     <collision>
@@ -61,6 +65,7 @@
       <material name="red" />
     </visual>
-    <xacro:cylinder_center_inertial mass="${pole_mass}" radius="${pole_radius}" length="${pole_length}" />
+    <xacro:cylinder_center_inertia mass="${pole_mass}" radius="${pole_radius}" length="${pole_length}" />
   </link>
+  <!--JOINT Pole_arm-->
   <joint name="pole_arm_joint" type="revolute">
     <parent link="pole_link"/>
@@ -70,4 +75,5 @@
     <limit effort="1000" lower="-2.5" upper="2.5" velocity="0.6" />
   </joint>
+  <!--Arm-->
   <link name="arm_link">
      <collision>
@@ -84,5 +90,26 @@
       <material name="orange" />
     </visual>
-    <xacro:cylinder_end_inertial mass="${arm_mass}" radius="${arm_radius}" length="${arm_length}" />
+    <xacro:cylinder_end_inertia mass="${arm_mass}" radius="${arm_radius}" length="${arm_length}" />
   </link>
+  <!--Transmissions-->
+  <transmission name="tran0">
+    <type>transmission_interface/SimpleTransmission</type>
+    <joint name="base_pole_joint">
+      <hardwareInterface>PositionJointInterface</hardwareInterface>
+    </joint>
+    <actuator name="motor0">
+      <hardwareInterface>PositionJointInterfce</hardwareInterface>
+      <mechanicalReduction>1</mechanicalReduction>
+    </actuator>
+  </transmission>
+  <transmission name="tran1">
+    <type>transmission_interface/SimpleTransmission</type>
+    <joint name="pole_arm_joint">
+      <hardwareInterface>PositionJointInterface</hardwareInterface>
+    </joint>
+    <actuator name="motor1">
+      <hardwareInterface>PositionJointInterfce</hardwareInterface>
+      <mechanicalReduction>1</mechanicalReduction>
+    </actuator>
+  </transmission>
 </robot>

File: robot/kai_description/urdf/kai.xacro (robot description, xacro)
@@ -16,5 +16,10 @@
   <xacro:property name="arm_mass" value="10.597" />
   <xacro:include filename="$(find kai_description)/urdf/kai.gazebo" />
+  <xacro:include filename="$(find kai_description)/urdf/macros.xacro" />
   <xacro:include filename="$(find kai_description)/urdf/materials.xacro" />
   <xacro:include filename="$(find kai_description)/urdf/geometry.xacro" />
+  <!--load ros_control plugin-->
+  <gazebo>
+    <plugin name="control" filename="libgazebo_ros_control.so"/>
+  </gazebo>
 </robot>
